Commit message: Added dummy camera link and joint

File: simulation_ws/src/i214_description/urdf/i214.xacro (robot description, xacro)
@@ -89,4 +89,15 @@
     </inertial>
   </link>
+  <!-- generate an optical frame http://www.ros.org/reps/rep-0103.html#suffix-frames
+      so that ros and opencv can operate on the camera frame correctly -->
+  <joint name="camera_optical_joint" type="fixed">
+    <!-- these values have to be these values otherwise the gazebo camera image
+        won't be aligned properly with the frame it is supposedly originating from -->
+    <origin xyz="0 0 0" rpy="${-pi/2} 0 ${-pi/2}"/>
+    <parent link="camera_link"/>
+    <child link="camera_link_optical"/>
+  </joint>
+  <link name="camera_link_optical">
+  </link>
   <link name="sensor_laser">
   <inertial>

Commit message: changed laser-scan height
changed visual property of sensor_laser to prevent blocking of camera view

File: simulation_ws/src/i214_description/urdf/i214.xacro (robot description, xacro)
@@ -109,5 +109,5 @@
       <origin xyz="0 0 0" rpy="0 0 0" />
       <geometry>
-      <cylinder radius="0.05" length="0.1"/>
+      <cylinder radius="0.05" length="0.03"/>
       </geometry>
       <material name="white" />

Commit message: Update i214.xacro
Updated for stable arc movement

File: simulation_ws/src/i214_description/urdf/i214.xacro (robot description, xacro)
@@ -28,5 +28,5 @@
     <collision name="collision_camera_mount">
       <geometry>
-        <box size="0.1 0.3 0.1"/>
+        <box size="0.1 0.25 0.1"/>
       </geometry>
     </collision>
@@ -34,5 +34,5 @@
       <origin rpy="0 0 0" xyz="0 0 0.05"/>
       <geometry>
-        <box size="0.1 0.3 0.1"/>
+        <box size="0.1 0.25 0.1"/>
       </geometry>
       <material name="blue"/>
@@ -89,20 +89,9 @@
     </inertial>
   </link>
-  <!-- generate an optical frame http://www.ros.org/reps/rep-0103.html#suffix-frames
-      so that ros and opencv can operate on the camera frame correctly -->
-  <joint name="camera_optical_joint" type="fixed">
-    <!-- these values have to be these values otherwise the gazebo camera image
-        won't be aligned properly with the frame it is supposedly originating from -->
-    <origin xyz="0 0 0" rpy="${-pi/2} 0 ${-pi/2}"/>
-    <parent link="camera_link"/>
-    <child link="camera_link_optical"/>
-  </joint>
-  <link name="camera_link_optical">
-  </link>
   <link name="sensor_laser">
   <inertial>
       <origin xyz="0 0 0" rpy="0 0 0" />
-      <mass value="1" />
-      <xacro:cylinder_inertia mass="1" r="0.05" l="0.1" />
+      <mass value="0.1" />
+      <xacro:cylinder_inertia m="0.1" r="0.05" h="0.1" />
   </inertial>
   <visual>
@@ -151,7 +140,67 @@
   </collision>
  </link>
-  <xacro:link_wheel name="link_right_wheel" />
-  <xacro:joint_wheel name="joint_right_wheel" child="link_right_wheel" origin_xyz="-0.05 0.15 0" />
-  <xacro:link_wheel name="link_left_wheel" />
-  <xacro:joint_wheel name="joint_left_wheel" child="link_left_wheel" origin_xyz="-0.05 -0.15 0" />
+ <link name="left_wheel">
+   <!--origin xyz="0.1 0.13 0.1" rpy="0 1.5707 1.5707"/-->
+   <collision name="collision">
+     <origin xyz="0 0 0" rpy="0 1.5707 1.5707"/>
+     <geometry>
+       <cylinder radius="0.1" length="0.05"/>
+     </geometry>
+   </collision>
+   <visual name="left_wheel_visual">
+     <origin xyz="0 0 0" rpy="0 1.5707 1.5707"/>
+     <geometry>
+       <cylinder radius="0.1" length="0.05"/>
+     </geometry>
+   </visual>
+   <inertial>
+     <origin xyz="0 0 0" rpy="0 1.5707 1.5707"/>
+     <mass value="5"/>
+     <cylinder_inertia m="5" r="0.1" h="0.05"/>
+     <inertia
+       ixx="1.0" ixy="0.0" ixz="0.0"
+       iyy="1.0" iyz="0.0"
+       izz="1.0"/>
+   </inertial>
+ </link>
+ <link name="right_wheel">
+   <!--origin xyz="0.1 -0.13 0.1" rpy="0 1.5707 1.5707"/-->
+   <collision name="collision">
+     <origin xyz="0 0 0" rpy="0 1.5707 1.5707"/>
+     <geometry>
+       <cylinder radius="0.1" length="0.05"/>
+     </geometry>
+   </collision>
+   <visual name="right_wheel_visual">
+     <origin xyz="0 0 0" rpy="0 1.5707 1.5707"/>
+     <geometry>
+       <cylinder radius="0.1" length="0.05"/>
+     </geometry>
+   </visual>
+   <inertial>
+     <origin xyz="0 0 0" rpy="0 1.5707 1.5707"/>
+     <mass value="5"/>
+     <cylinder_inertia m="5" r="0.1" h="0.05"/>
+     <inertia
+       ixx="1.0" ixy="0.0" ixz="0.0"
+       iyy="1.0" iyz="0.0"
+       izz="1.0"/>
+   </inertial>
+ </link>
+ <joint type="continuous" name="left_wheel_hinge">
+   <origin xyz="-0.1 0.15 0" rpy="0 0 0"/>
+   <child link="left_wheel"/>
+   <parent link="link_chassis"/>
+   <axis xyz="0 1 0" rpy="0 0 0"/>
+   <limit effort="100" velocity="100"/>
+   <joint_properties damping="0.0" friction="0.0"/>
+ </joint>
+ <joint type="continuous" name="right_wheel_hinge">
+   <origin xyz="-0.1 -0.15 0" rpy="0 0 0"/>
+   <child link="right_wheel"/>
+   <parent link="link_chassis"/>
+   <axis xyz="0 1 0" rpy="0 0 0"/>
+   <limit effort="100" velocity="100"/>
+   <joint_properties damping="0.0" friction="0.0"/>
+ </joint>
 </robot>

Commit message: Added transmission tags for movement of camera joint

File: simulation_ws/src/i214_description/urdf/i214.xacro (robot description, xacro)
@@ -62,9 +62,12 @@
     </visual>
   </link>
-  <joint name="camera_joint" type="fixed">
-    <axis xyz="0 1 0" />
+  <joint name="camera_joint" type="continuous">
+    <!--<limit upper="1.57" lower="-1.57" velocity="10" effort="1"/>-->
+    <axis xyz="0 0 1" />
     <origin xyz="0 0 0.15" rpy="0 0 0"/>
     <parent link="link_chassis"/>
     <child link="camera_link"/>
+    <limit effort="100" velocity="100"/>
+   <!--<joint_properties damping="0.0" friction="0.0"/>-->
   </joint>
   <!-- Camera -->
@@ -204,3 +207,14 @@
    <joint_properties damping="0.0" friction="0.0"/>
  </joint>
+   <!-- transmission -->
+    <transmission name="tran1">
+    <type>transmission_interface/SimpleTransmission</type>
+    <joint name="camera_joint">
+      <hardwareInterface>hardware_interface/VelocityJointInterface</hardwareInterface>
+    </joint>
+    <actuator name="motor1">
+      <hardwareInterface>hardware_interface/VelocityJointInterface</hardwareInterface>
+      <mechanicalReduction>1</mechanicalReduction>
+    </actuator>
+  </transmission>
 </robot>
